File: kicad/uart-rs232-rs485.kicad_sch (KiCad schematic)
At the start: 21 parts, among them U4 MAX3232, U5 YD3082EESA

Commit message: created bom for order lcsc
Parts:
- C16, C17, C18, C19, C20, C21, D8, D9, R26, R27, R28, R29, R30, R31, R32, U4, U5: now not fitted; now left out of the parts list
